File: gvifhat.kicad_sch (KiCad schematic)
At the start: 66 parts, among them J1 Raspberry_Pi_2_3, J2 GVIFout, J3 GVIFin, J4 USB_A, J5 USB_A, J6 touch_IN, J7 touch_OUT, J8 Conn_01x02_Pin, J9 UPDI, U1 CXB1457R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

Commit message: replaced solder-in battery with a cr1220 holder
Parts:
- BT1: footprint Battery:Battery_Panasonic_CR1220-VCN_Vertical_CircularHoles -> hdmi2lvds:MPD_BC501SM-TR
